File: 555-Oscilador-pisca-r01.kicad_pcb (KiCad board)
At the start: 2 copper layers, 49.5 x 49.3 mm, 10 parts, among them J1 Saída Piscante, J2 Alimentação, U1 NE555

Commit message: backups
Other:
- net class Default removed
